File: 1-WireWeMos.sch (EAGLE design)
At the start: 18 parts, among them IC1 DS2482-100, J2 RJ11-6PTH, Q1 BSS84, Q2 BSS138, Q3 BSS138, X1 RJ45-6L-B, X2 TERMINAL-BLOCK-3.5MM-3-PIN-RO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

Commit message: year number fixed
Other:
- note added: "V1 (2018-04-22)"
- note removed: "V1 (2019-04-22)"
Changed lines of the file:
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@@
 <text x="7.62" y="6.858" size="1.778" layer="94">SKU: ow1</text>
 <text x="7.62" y="12.7" size="2.794" layer="94">1-Wire WeMos</text>
-<text x="81.28" y="6.858" size="1.778" layer="94">V1 (2019-04-22)</text>
+<text x="81.28" y="6.858" size="1.778" layer="94">V1 (2018-04-22)</text>
 <text x="32.766" y="6.858" size="1.778" layer="94">taaralabs.eu/ow1</text>
 <frame x1="5.08" y1="5.08" x2="109.22" y2="17.78" columns="0" rows="0" layer="94" border-left="no" border-top="no" border-right="no" border-bottom="no"/>
